File: hardware/control_driver/control_driver.sch (EAGLE design)
At the start: 2 parts, among them IC1 STM32F030K6T6

Commit message: Допиливается котроллер управления
Connections:
- new net DATA0: IC1MCU.PA0-WKUP
- new net DATA1: IC1MCU.PA1
- new net DATA2: IC1MCU.PA2
- new net DATA3: IC1MCU.PA3
- new net DATA4: IC1MCU.PA4
- new net DATA5: IC1MCU.PA5
- new net DATA6: IC1MCU.PA6
- new net DATA7: IC1MCU.PA7
- new net E: IC1MCU.PA8
- new net GND: HG1.K
- new net PWM1: IC1MCU.PB1
- new net PWM2: IC1MCU.PB0
- new net RS: IC1MCU.PA11
- new net RW: IC1MCU.PA12
- new net SWDCLK: IC1MCU.PA14
- new net SWDIO: IC1MCU.PA13
- new net UART_RX: IC1MCU.PA10
- new net UART_TX: IC1MCU.PA9
Changed lines of the file:
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@@
 </instances>
 <busses>
+<bus name="DATA0,DATA1,DATA2,DATA3,DATA4,DATA5,DATA6,DATA7,E,RS,RW,UART_TX,UART_RX,SWDIO,SWDCLK,LED1,LED2,LED3,PWM1,PWM2,VCC_3.3V,VCC_5V,GND">
+<segment>
+<wire x1="223.52" y1="121.92" x2="223.52" y2="233.68" width="0.762" layer="92"/>
+<wire x1="223.52" y1="233.68" x2="86.36" y2="233.68" width="0.762" layer="92"/>
+</segment>
+</bus>
 </busses>
 <nets>
+<net name="DATA0" class="0">
+<segment>
+<pinref part="IC1" gate="MCU" pin="PA0-WKUP"/>
+<wire x1="223.52" y1="127" x2="208.28" y2="127" width="0.1524" layer="91"/>
+<label x="217.17" y="127.508" size="1.27" layer="95" font="vector"/>
+</segment>
+</net>
+<net name="DATA1" class="0">
+<segment>
+<pinref part="IC1" gate="MCU" pin="PA1"/>
+<wire x1="223.52" y1="129.54" x2="208.28" y2="129.54" width="0.1524" layer="91"/>
+<label x="217.17" y="130.048" size="1.27" layer="95" font="vector"/>
+</segment>
+</net>
+<net name="DATA2" class="0">
+<segment>
+<pinref part="IC1" gate="MCU" pin="PA2"/>
+<wire x1="223.52" y1="132.08" x2="208.28" y2="132.08" width="0.1524" layer="91"/>
+<label x="217.17" y="132.588" size="1.27" layer="95" font="vector"/>
+</segment>
+</net>
+<net name="DATA3" class="0">
+<segment>
+<pinref part="IC1" gate="MCU" pin="PA3"/>
+<wire x1="223.52" y1="134.62" x2="208.28" y2="134.62" width="0.1524" layer="91"/>
+<label x="217.17" y="135.128" size="1.27" layer="95" font="vector"/>
+</segment>
+</net>
+<net name="DATA4" class="0">
+<segment>
+<pinref part="IC1" gate="MCU" pin="PA4"/>
+<wire x1="223.52" y1="137.16" x2="208.28" y2="137.16" width="0.1524" layer="91"/>
+<label x="217.17" y="137.668" size="1.27" layer="95" font="vector"/>
+</segment>
+</net>
+<net name="DATA5" class="0">
+<segment>
+<pinref part="IC1" gate="MCU" pin="PA5"/>
+<wire x1="223.52" y1="139.7" x2="208.28" y2="139.7" width="0.1524" layer="91"/>
+<label x="217.17" y="140.208" size="1.27" layer="95" font="vector"/>
+</segment>
+</net>
+<net name="DATA6" class="0">
+<segment>
+<pinref part="IC1" gate="MCU" pin="PA6"/>
+<wire x1="223.52" y1="142.24" x2="208.28" y2="142.24" width="0.1524" layer="91"/>
+<label x="217.17" y="142.748" size="1.27" layer="95" font="vector"/>
+</segment>
+</net>
+<net name="DATA7" class="0">
+<segment>
+<pinref part="IC1" gate="MCU" pin="PA7"/>
+<wire x1="223.52" y1="144.78" x2="208.28" y2="144.78" width="0.1524" layer="91"/>
+<label x="217.17" y="145.288" size="1.27" layer="95" font="vector"/>
+</segment>
+</net>
+<net name="E" class="0">
+<segment>
+<pinref part="IC1" gate="MCU" pin="PA8"/>
+<wire x1="223.52" y1="147.32" x2="208.28" y2="147.32" width="0.1524" layer="91"/>
+<label x="220.98" y="147.828" size="1.27" layer="95" font="vector"/>
+</segment>
+</net>
+<net name="RS" class="0">
+<segment>
+<pinref part="IC1" gate="MCU" pin="PA11"/>
+<wire x1="223.52" y1="154.94" x2="208.28" y2="154.94" width="0.1524" layer="91"/>
+<label x="220.472" y="155.448" size="1.27" layer="95" font="vector"/>
+</segment>
+</net>
+<net name="RW" class="0">
+<segment>
+<pinref part="IC1" gate="MCU" pin="PA12"/>
+<wire x1="223.52" y1="157.48" x2="208.28" y2="157.48" width="0.1524" layer="91"/>
+<label x="220.472" y="157.988" size="1.27" layer="95" font="vector"/>
+</segment>
+</net>
+<net name="UART_TX" class="0">
+<segment>
+<pinref part="IC1" gate="MCU" pin="PA9"/>
+<wire x1="223.52" y1="149.86" x2="208.28" y2="149.86" width="0.1524" layer="91"/>
+<label x="214.884" y="150.368" size="1.27" layer="95" font="vector"/>
+</segment>
+</net>
+<net name="UART_RX" class="0">
+<segment>
+<pinref part="IC1" gate="MCU" pin="PA10"/>
+<wire x1="223.52" y1="152.4" x2="208.28" y2="152.4" width="0.1524" layer="91"/>
+<label x="214.884" y="152.908" size="1.27" layer="95" font="vector"/>
+</segment>
+</net>
+<net name="GND" class="0">
+<segment>
+<pinref part="HG1" gate="G$1" pin="K"/>
+<wire x1="241.3" y1="121.92" x2="223.52" y2="121.92" width="0.1524" layer="91"/>
+<label x="224.536" y="122.428" size="1.27" layer="95" font="vector"/>
+</segment>
+</net>
+<net name="SWDIO" class="0">
+<segment>
+<pinref part="IC1" gate="MCU" pin="PA13"/>
+<wire x1="223.52" y1="160.02" x2="208.28" y2="160.02" width="0.1524" layer="91"/>
+<label x="217.424" y="160.528" size="1.27" layer="95" font="vector"/>
+</segment>
+</net>
+<net name="SWDCLK" class="0">
+<segment>
+<pinref part="IC1" gate="MCU" pin="PA14"/>
+<wire x1="223.52" y1="162.56" x2="208.28" y2="162.56" width="0.1524" layer="91"/>
+<label x="215.9" y="163.068" size="1.27" layer="95" font="vector"/>
+</segment>
+</net>
+<net name="PWM1" class="0">
+<segment>
+<pinref part="IC1" gate="MCU" pin="PB1"/>
+<wire x1="223.52" y1="172.72" x2="208.28" y2="172.72" width="0.1524" layer="91"/>
+<label x="218.44" y="173.228" size="1.27" layer="95" font="vector"/>
+</segment>
+</net>
+<net name="PWM2" class="0">
+<segment>
+<pinref part="IC1" gate="MCU" pin="PB0"/>
+<wire x1="223.52" y1="170.18" x2="208.28" y2="170.18" width="0.1524" layer="91"/>
+<label x="218.44" y="170.688" size="1.27" layer="95" font="vector"/>
+</segment>
+</net>
 </nets>
 </sheet>

Commit message: Добавлена трассиворка платы управления
Parts:
- added C1, C17, C18: 33u, rcl:CPOL-EUSMCB
- added C10, C15, C25, C6: 10u, rcl:CPOL-EUSMCA
- added C11, C12, C13, C14, C16, C19, C20, C21, C24, C26, C27, C4, C5, C7: 0.1u, rcl:C-EUC0603
- added C2, C3, C8, C9: 33u, rcl:CPOL-EUSMCC
- added C22, C23: 20p, rcl:C-EUC0603
- added IC2, IC3: ADuM1250ARZ, onega:ADUM1250
- added IC4, IC5: LM317LD, linear:LM317LD
- added IC6: CP2102, silabs:CP2102
- added IC7: AT24C512, onega:24C512
- added IC8: STM32F051K8U6, micro-stm_v3:STM32F051K8U
- added J1: 22-27-2041-04, con-molex:22-27-2041-04
- added J2: 22-27-2031-03, con-molex:22-27-2031-03
- added JP1: (no value), pinhead:PINHD-1X55X2MM
- added JP2, JP3, JP4: (no value), pinhead:PINHD-1X2
- added L1, L2, L3, L4, L5: 100uH, rcl:L-US
- added LED1: USB ON, led:LEDCHIPLED_0805
- added R1, R10, R12, R13, R16, R17, R18, R3, R4, R5, R9: 10k, rcl:R-EU_R0603
- added R11, R6: 20, rcl:R-EU_R0603
- added R14, R15: 1k, rcl:R-EU_R0603
- added R19: 560, rcl:R-EU_R0603
- added R2: 1M, rcl:R-EU_R0603
- added R20: 1k, rcl:R-TRIMM4G/J
- added R21, R22: 4.7k, rcl:R-EU_R0603
- added R23: 120, rcl:R-EU_R0805
- added R7: 1.5k, rcl:R-EU_R0603
- added R8: 3k, rcl:R-EU_R0603
- added X1: (no value), con-hirose:MICRO-USB
- added Z1: 8MHz, onega:CRYSTAL_5X7MM
- IC1: value STM32F030K6T6 -> USB6B1; device micro-stm_v3:STM32F030K6T -> st-microelectronics:USB6B1
Connections:
- new net !SD: IC3.SCL2, IC8MCU.PA15, R13.2
- new net CONTRAST: HG1.VO, R20.S
- new net I2C_SCL: IC7.SCL, IC8MCU.PB6, R22.2
- new net I2C_SDA: IC7.SDA, IC8MCU.PB7, R21.2
- new net LED: IC8MCU.PA12
- new net N$1: HG1.A, R23.2
- new net N$10: IC4.ADJ, R14.1, R7.2
- new net N$11: C12.2, C8.+, IC4.VI, L1.2
- new net N$12: IC5.ADJ, R15.1, R8.2
- new net N$13: C1.+, R2.2, X1.SHD@1, X1.SHD@2, X1.SHD@3, X1.SHD@4
- new net N$14: IC1.IO1, X1.D+
- new net N$15: IC1.IO2, X1.D-
- new net N$16: IC1.GND, X1.GND
- new net N$17: C6.+, C7.1, IC1.VCC, X1.VCC
- new net N$18: C22.1, IC8MCU.OSC_OUT, Z1.1
- new net N$19: C23.1, IC8MCU.OSC_IN, Z1.2
- new net N$2: IC1.IO2@2, R6.1
- new net N$20: C24.2, C25.+, IC7.VCC, L5.1
- new net N$21: IC8MCU.NRST, R16.2
- new net N$24: IC2.VDD1, IC3.VDD1, JP1.5
- new net N$25: IC8MCU.BOOT0, R18.2
- new net N$26: IC2.SCL1, JP2.1, R1.2
- new net N$27: IC2.SDA1, JP1.1, R3.2
- new net N$28: IC3.SDA1, JP1.3, R5.2
- new net N$29: IC3.SCL1, JP1.4, R4.2
- new net N$3: IC1.IO1@2, R11.1
- new net N$30: IC2.GND1, IC3.GND1, JP1.2, JP2.2, R1.1, R3.1, R4.1, R5.1
- new net N$4: IC6.D-, R6.2
- new net N$5: IC6.D+, R11.2
- new net N$6: LED1.A, R19.1
- new net N$7: C10.+, C11.1, IC1.VCC@2, IC6.REGIN, IC6.VBUS
- new net N$8: IC6.!RST, R17.1
- new net N$9: IC6.SUSPEND, LED1.C
- new net POL: IC3.SDA2, IC8MCU.PA8, R10.2
- new net POWER_ON: IC8MCU.PA11, JP4.1
- new net TEM_SENS_RX: IC8MCU.PA10, J2-2.S
- new net TEM_SENS_TX: IC8MCU.PA9, J2-1.S
- new net VCC_12V: C2.+, C3.+, C4.2, C5.2, JP3.1, L1.1, L2.1
- new net VCC_12V_IN: C13.2, C9.+, IC5.VI, L2.2
- new net VCC_3.3V: C14.1, C15.+, C16.1, C21.2, C26.2, C27.2, HG1.VDD, IC2.VDD2, IC3.VDD2, IC6.VDD, IC8MCU.VDDA, IC8PWR.VDD@1, IC8PWR.VDD@2, J1-1.S, L3.2, L5.2, R16.1, R17.2, R19.2, R20.E, R21.1, R22.1
- new net VCC_3.3V1: C18.+, C20.2, IC5.VO, IC5.VO@1, IC5.VO@2, IC5.VO@3, L4.1, R15.2
- new net VCC_3.3V2222: C17.+, C19.2, IC4.VO, IC4.VO@1, IC4.VO@2, IC4.VO@3, L3.1, R14.2
- new net VCC_5V: L4.2, R23.1
- net DATA0: now also HG1.DB0, IC8MCU.PA4; no longer IC1MCU.PA0-WKUP
- net DATA1: now also HG1.DB1, IC8MCU.PA5; no longer IC1MCU.PA1
- net DATA2: now also HG1.DB2, IC8MCU.PA6; no longer IC1MCU.PA2
- net DATA3: now also HG1.DB3, IC8MCU.PA7; no longer IC1MCU.PA3
- net DATA4: now also HG1.DB4, IC8MCU.PB2; no longer IC1MCU.PA4
- net DATA5: now also HG1.DB5, IC8MCU.PB3; no longer IC1MCU.PA5
- net DATA6: now also HG1.DB6, IC8MCU.PB4; no longer IC1MCU.PA6
- net DATA7: now also HG1.DB7, IC8MCU.PB5; no longer IC1MCU.PA7
- net E: now also HG1.E, IC8MCU.PB1; no longer IC1MCU.PA8
- net GND: now also C1.-, C10.-, C11.2, C12.1, C13.1, C14.2, C15.-, C16.2, C17.-, C18.-, C19.1, C2.-, C20.1, C21.1, C22.2, C23.2, C24.1, C25.-, C26.1, C27.1, C3.-, C4.1, C5.1, C6.-, C7.2, C8.-, C9.-, HG1.VSS, IC1.GND@2, IC2.GND2, IC3.GND2, IC6.GND, IC6.GND@EXP, IC6.GND@M, IC7.A0, IC7.A1, IC7.GND, IC8PWR.VSS@1, J1-4.S, J2-3.S, JP3.2, JP4.2, R10.1, R12.1, R13.1, R18.1, R2.1, R20.A, R7.1, R8.1, R9.1
- net PWM1: now also IC2.SDA2, IC8MCU.PA1, R9.2; no longer IC1MCU.PB1
- net PWM2: now also IC2.SCL2, IC8MCU.PB8, R12.2; no longer IC1MCU.PB0
- net RS: now also HG1.RS, IC8MCU.PB0; no longer IC1MCU.PA11
- net RW: now also HG1.R/W, IC8MCU.PA0-WKUP; no longer IC1MCU.PA12
- net SWDCLK: now also IC8MCU.PA14, J1-2.S; no longer IC1MCU.PA14
- net SWDIO: now also IC8MCU.PA13, J1-3.S; no longer IC1MCU.PA13
- net UART_RX: now also IC6.TXD, IC8MCU.PA3; no longer IC1MCU.PA10
- net UART_TX: now also IC6.RXD, IC8MCU.PA2; no longer IC1MCU.PA9
Other:
- moved on the sheet: HG1
