File: hardware/h_bridge_driver/h_bridge_driver.brd (EAGLE design)
At the start: 90 x 35 mm, 42 parts, among them IC1 IR2184S, IC2 78L05SMD, IC3 SN74HC02PW, IC4 IR2184S, Q1 IRF540, Q2 IRF540, Q3 IRF540, Q4 IRF540

Commit message: Добавлена трассиворка платы управления
Parts:
- removed JP1: (no value), pinhead:1X04
- added JP2: (no value), pinhead:1_05X2MM
- moved L4 4.27 mm to (66.2, 10.0), turned to 180 degrees
- moved R7 2.85 mm to (60.5, 11.2), turned to 270 degrees
- moved C10 1.41 mm to (66.5, 22.0)
- moved C2 0.87 mm to (29.7, 25.3)
Connections:
- removed net !DRIVER_EN: IC4.2, R9.2
- removed net N$21: IC1.2, R2.2
- new net !SD: IC1.2, IC4.2, JP2.4, R2.2, R9.2
- net +5V_VS: now also JP2.5
- net GND: now also JP2.2; no longer JP1.2
- net N$12: now also JP2.1; no longer JP1.1
- net N$9: now also JP2.3; no longer JP1.3
Routing:
- net !SD: track 0.00 -> 121.9 mm, vias 0 -> 5
- net +5V_VS: track 19.0 -> 46.3 mm, vias 2 -> 4
- net GND: track 194.4 -> 170.4 mm
- net N$9: track 25.9 -> 32.9 mm, vias 0 -> 1
- net N$17: track 15.0 -> 21.1 mm, vias 0 -> 2
- net N$13: track 10.6 -> 8.31 mm
- net N$21: track 2.05 -> 0.00 mm
- net N$7: track 5.06 -> 6.96 mm
- net !DRIVER_EN: track 1.74 -> 0.00 mm
- net +12V_VS: track 151.9 -> 150.2 mm
- net N$12: track 29.5 -> 30.5 mm
- net PWM2: track 67.2 -> 66.2 mm
- net N$18: track 74.0 -> 74.9 mm
- net N$8: track 26.4 -> 27.2 mm
Other:
- board text added: "Created by Sergey Sklyarov Nikolay Kuznetsov"
- board text added: "H Bridge driver"
- board text added: "Saratov State University"
- board text added: "Saratov, 2015-2016"
