File: hardware/h_bridge_driver/h_bridge_driver.sch (EAGLE design)
At the start: 38 parts, among them IC1 IR2184S, IC2 78L05SMD, IC3 SN74HC02PW, IC4 IR2184S, Q1 IRF540, Q2 IRF540, Q3 IRF540, Q4 IRF540, X1 MKDSN1,5/2-5,08, X2 MKDSN1,5/3-5,08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

Commit message: Добавлена трассиворка платы управления
Parts:
- removed JP1: (no value), pinhead:PINHD-1X4
- added JP2: (no value), pinhead:PINHD-1X55X2MM
Connections:
- removed net !DRIVER_EN: IC4.!SD, R9.2
- removed net N$21: IC1.!SD, R2.2
- new net !SD: IC1.!SD, IC4.!SD, JP2.4, R2.2, R9.2
- net +5V_VS: now also JP2.5
- net GND: now also JP2.2; no longer JP1.2
- net N$12: now also JP2.1; no longer JP1.1
- net N$9: now also JP2.3; no longer JP1.3
Changed lines of the file:
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@@
 <setting verticaltext="up"/>
 </settings>
-<grid distance="0.1" unitdist="inch" unit="inch" style="lines" multiple="1" display="yes" altdistance="0.01" altunitdist="inch" altunit="inch"/>
+<grid distance="0.1" unitdist="inch" unit="inch" style="lines" multiple="1" display="no" altdistance="0.01" altunitdist="inch" altunit="inch"/>
 <layers>
 <layer number="1" name="Top" color="4" fill="1" visible="no" active="no"/>
@@
 <part name="GND8" library="supply1" deviceset="GND" device=""/>
 <part name="GND9" library="supply1" deviceset="GND" device=""/>
-<part name="JP1" library="pinhead" deviceset="PINHD-1X4" device=""/>
+<part name="JP2" library="pinhead" deviceset="PINHD-1X5" device="5X2MM"/>
 </parts>
 <sheets>
@@
 <instance part="GND8" gate="1" x="121.92" y="116.84"/>
 <instance part="GND9" gate="1" x="132.08" y="116.84"/>
-<instance part="JP1" gate="A" x="78.74" y="132.08" rot="MR0"/>
+<instance part="JP2" gate="A" x="78.74" y="132.08" rot="MR0"/>
 </instances>
 <busses>
@@
 <wire x1="96.52" y1="134.62" x2="96.52" y2="119.38" width="0.1524" layer="91"/>
 <pinref part="GND6" gate="1" pin="GND"/>
-<pinref part="JP1" gate="A" pin="2"/>
+<pinref part="JP2" gate="A" pin="2"/>
 </segment>
 <segment>
@@
 </segment>
 </net>
-<net name="!DRIVER_EN" class="0">
-<segment>
-<pinref part="IC4" gate="G$1" pin="!SD"/>
-<pinref part="R9" gate="G$1" pin="2"/>
-<wire x1="177.8" y1="78.74" x2="182.88" y2="78.74" width="0.1524" layer="91"/>
-<wire x1="182.88" y1="78.74" x2="182.88" y2="60.96" width="0.1524" layer="91"/>
-</segment>
-</net>
 <net name="N$9" class="0">
 <segment>
@@
 <wire x1="132.08" y1="129.54" x2="132.08" y2="132.08" width="0.1524" layer="91"/>
 <junction x="132.08" y="132.08"/>
-<pinref part="JP1" gate="A" pin="3"/>
+<pinref part="JP2" gate="A" pin="3"/>
 </segment>
 </net>
@@
 <wire x1="121.92" y1="129.54" x2="121.92" y2="137.16" width="0.1524" layer="91"/>
 <junction x="121.92" y="137.16"/>
-<pinref part="JP1" gate="A" pin="1"/>
+<pinref part="JP2" gate="A" pin="1"/>
 </segment>
 </net>
@@
 <label x="205.74" y="149.86" size="1.778" layer="95" xref="yes"/>
 </segment>
-</net>
-<net name="N$21" class="0">
+<segment>
+<pinref part="JP2" gate="A" pin="5"/>
+<wire x1="81.28" y1="127" x2="88.9" y2="127" width="0.1524" layer="91"/>
+<wire x1="88.9" y1="127" x2="88.9" y2="124.46" width="0.1524" layer="91"/>
+<label x="88.9" y="124.46" size="1.778" layer="95" rot="R270" xref="yes"/>
+</segment>
+</net>
+<net name="!SD" class="0">
 <segment>
 <pinref part="IC1" gate="G$1" pin="!SD"/>
@@
 <pinref part="R2" gate="G$1" pin="2"/>
 <wire x1="50.8" y1="68.58" x2="50.8" y2="78.74" width="0.1524" layer="91"/>
-</segment>
-</net>
+<wire x1="38.1" y1="78.74" x2="50.8" y2="78.74" width="0.1524" layer="91"/>
+<junction x="50.8" y="78.74"/>
+<label x="38.1" y="78.74" size="1.778" layer="95" rot="R180" xref="yes"/>
+</segment>
+<segment>
+<pinref part="IC4" gate="G$1" pin="!SD"/>
+<pinref part="R9" gate="G$1" pin="2"/>
+<wire x1="177.8" y1="78.74" x2="182.88" y2="78.74" width="0.1524" layer="91"/>
+<wire x1="182.88" y1="78.74" x2="182.88" y2="60.96" width="0.1524" layer="91"/>
+<wire x1="182.88" y1="78.74" x2="195.58" y2="78.74" width="0.1524" layer="91"/>
+<label x="195.58" y="78.74" size="1.778" layer="95" xref="yes"/>
+<junction x="182.88" y="78.74"/>
+</segment>
+<segment>
+<wire x1="81.28" y1="129.54" x2="93.98" y2="129.54" width="0.1524" layer="91"/>
+<wire x1="93.98" y1="124.46" x2="93.98" y2="129.54" width="0.1524" layer="91"/>
+<label x="93.98" y="124.46" size="1.778" layer="95" rot="R270" xref="yes"/>
+<pinref part="JP2" gate="A" pin="4"/>
+</segment>
+</net>
